File: kicad/attiny13_breakout/attiny13_breakout.kicad_pcb (KiCad board)
At the start: 2 copper layers, 50.8 x 25.4 mm, 22 parts, among them J1 Pwr OUT, J2 Power, J3 Alt IN, J4 Conn_01x04_Male, J5 Conn_01x04_Male, J6 ISP, SW1 B3S-1000, U1 TC1262-33, U2 ATtiny13-20S

Commit message: Net correction for Rev 1.1
Connections:
- C3 pad 1: /~{RESET} -> /PB5_RESET
- D4 pad 2: /~{RESET} -> /PB5_RESET
- R1 pad 2: /~{RESET} -> /PB5_RESET
- SW1 pad 1: /~{RESET} -> /PB5_RESET
- U2 pad 1: /~{RESET} -> /PB5_RESET
Routing:
- net /PB5_RESET: track 25.2 -> 55.4 mm
- net /~{RESET}: track 23.7 -> 0.00 mm
Other:
- board text added: "ATTiny13 Breakout Rev 1.1"
- board text removed: "ATTiny13 Breakout Rev 1.0"
