File: kicad/attiny13_breakout/attiny13_breakout.kicad_sch (KiCad schematic)
At the start: 22 parts, among them J1 Pwr OUT, J2 Power, J3 Alt IN, J4 Conn_01x04_Male, J5 Conn_01x04_Male, J6 ISP, SW1 B3S-1000, U1 TC1262-33, U2 ATtiny13-20S

Commit message: Net correction for Rev 1.1
Connections:
- net ~{RESET} is gone; now on net PB5_RESET: C3.1, D4.2 (A), R1.2, SW1.1, U2.1 (~{RESET}/PB5)
Changed lines of the file:
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@@
     (effects (font (size 1.27 1.27)) (justify left bottom))
   )
-  (label "~{RESET}" (at 118.11 113.03 180)
+  (label "PB5_RESET" (at 118.11 113.03 180)
     (effects (font (size 1.27 1.27)) (justify right bottom))
   )
